Commit message: Update robot arm model and visualization

File: 6dof-robotic-arm/ros2_ws/src/six_dof_arm/urdf/arm.urdf.xacro (robot description, xacro)
@@ -7,163 +7,73 @@
   <xacro:property name="link3_length" value="0.12"/>
   <xacro:property name="link_radius" value="0.025"/>
-  <!-- Reusable cylindrical link geometry.
-       Cylinders are aligned along their local Z axes. -->
-  <xacro:macro name="cylinder_link" params="name length radius mass">
-    <link name="${name}">
-      <inertial>
-        <origin xyz="0 0 ${length / 2}" rpy="0 0 0"/>
-        <mass value="${mass}"/>
-        <inertia
-          ixx="${mass * (3 * radius * radius + length * length) / 12}"
-          ixy="0" ixz="0"
-          iyy="${mass * (3 * radius * radius + length * length) / 12}"
-          iyz="0"
-          izz="${mass * radius * radius / 2}"/>
-      </inertial>
-      <visual>
-        <origin xyz="0 0 ${length / 2}" rpy="0 0 0"/>
-        <geometry>
-          <cylinder radius="${radius}" length="${length}"/>
-        </geometry>
-        <material name="arm_blue">
-          <color rgba="0.2 0.45 0.85 1.0"/>
-        </material>
-      </visual>
-      <collision>
-        <origin xyz="0 0 ${length / 2}" rpy="0 0 0"/>
-        <geometry>
-          <cylinder radius="${radius}" length="${length}"/>
-        </geometry>
-      </collision>
-    </link>
-  </xacro:macro>
-  <!-- Base -->
+  <!-- Base 1: fixed base -->
   <link name="base_link">
     <visual>
-      <origin xyz="0 0 ${base_height / 2}"/>
+      <origin xyz="-0.077 -0.070 0" rpy="0 0 0"/>
       <geometry>
-        <cylinder radius="0.06" length="${base_height}"/>
+        <mesh filename="package://six_dof_arm/meshes/Base1.STL"
+              scale="0.001 0.001 0.001"/>
       </geometry>
-      <material name="base_gray">
-        <color rgba="0.35 0.35 0.38 1"/>
+    </visual>
+  </link>
+  <!-- Joint 1: rotating base -->
+  <link name="base2_link">
+    <visual>
+      <origin xyz="-0.06 -0.06 0.003" rpy="0 0 0"/>
+      <geometry>
+        <mesh filename="package://six_dof_arm/meshes/Base2.STL"
+              scale="0.001 0.001 0.001"/>
+      </geometry>
+      <material name="base2_blue">
+        <color rgba="0.15 0.35 0.8 1.0"/>
+    </material>
+    </visual>
+  </link>
+  <joint name="joint1" type="revolute">
+    <parent link="base_link"/>
+    <child link="base2_link"/>
+    <origin xyz="0 0 0.035" rpy="0 0 0"/>
+    <axis xyz="0 0 1"/>
+    <limit lower="-3.14159" upper="3.14159"
+          effort="10" velocity="1.0"/>
+  </joint>
+  <!-- Joint 2: first arm -->
+  <link name="link1">
+    <visual>
+      <origin xyz="-0.013 -0.022 -0.008" rpy="0 0 0"/>
+      <geometry>
+        <mesh filename="package://six_dof_arm/meshes/Link1.STL"
+              scale="0.001 0.001 0.001"/>
+      </geometry>
+    </visual>
+  </link>
+  <joint name="joint2" type="revolute">
+    <parent link="base2_link"/>
+    <child link="link1"/>
+    <origin xyz="0 0 0.025" rpy="0 0 0"/>
+    <axis xyz="0 1 0"/>
+    <limit lower="-1.5708" upper="1.5708"
+          effort="10" velocity="1.0"/>
+  </joint>
+  <!-- Joint 3: second arm -->
+  <link name="link2">
+    <visual>
+      <origin xyz="-0.0148 -0.0145 -0.009" rpy="0 0 0"/>
+      <geometry>
+        <mesh filename="package://six_dof_arm/meshes/Link2.STL"
+              scale="0.001 0.001 0.001"/>
+      </geometry>
+      <material name="base2_blue">
+        <color rgba="0.15 0.35 0.8 1.0"/>
       </material>
     </visual>
-    <collision>
-      <origin xyz="0 0 ${base_height / 2}"/>
-      <geometry>
-        <cylinder radius="0.06" length="${base_height}"/>
-      </geometry>
-    </collision>
-    <inertial>
-      <origin xyz="0 0 ${base_height / 2}"/>
-      <mass value="1.0"/>
-      <inertia ixx="0.002" ixy="0" ixz="0"
-               iyy="0.002" iyz="0" izz="0.003"/>
-    </inertial>
   </link>
-  <!-- Shoulder link: rotates about the vertical axis. -->
-  <xacro:cylinder_link name="link1" length="${link1_length}"
-                       radius="${link_radius}" mass="0.3"/>
-  <joint name="joint1" type="revolute">
-    <parent link="base_link"/>
-    <child link="link1"/>
-    <origin xyz="0 0 ${base_height}" rpy="0 0 0"/>
-    <axis xyz="0 0 1"/>
-    <limit lower="-3.14159" upper="3.14159"
-           effort="10" velocity="1.0"/>
-  </joint>
-  <xacro:cylinder_link name="link2" length="${link2_length}"
-                       radius="${link_radius}" mass="0.25"/>
-  <joint name="joint2" type="revolute">
+  <joint name="joint3" type="revolute">
     <parent link="link1"/>
     <child link="link2"/>
-    <origin xyz="0 0 ${link1_length}" rpy="0 0 0"/>
-    <axis xyz="0 1 0"/>
-    <limit lower="-1.5708" upper="1.5708"
-           effort="10" velocity="1.0"/>
-  </joint>
-  <xacro:cylinder_link name="link3" length="${link3_length}"
-                       radius="${link_radius}" mass="0.2"/>
-  <joint name="joint3" type="revolute">
-    <parent link="link2"/>
-    <child link="link3"/>
-    <origin xyz="0 0 ${link2_length}" rpy="0 0 0"/>
+    <origin xyz="0 0 0.095" rpy="0 0 0"/>
     <axis xyz="0 1 0"/>
     <limit lower="-2.0" upper="2.0"
-           effort="8" velocity="1.0"/>
-  </joint>
-  <!-- Wrist placeholders -->
-  <link name="wrist_link">
-    <visual>
-      <geometry><sphere radius="0.025"/></geometry>
-      <material name="wrist_gray">
-        <color rgba="0.7 0.7 0.72 1"/>
-      </material>
-    </visual>
-    <collision>
-      <geometry><sphere radius="0.025"/></geometry>
-    </collision>
-    <inertial>
-      <mass value="0.1"/>
-      <inertia ixx="0.0001" ixy="0" ixz="0"
-               iyy="0.0001" iyz="0" izz="0.0001"/>
-    </inertial>
-  </link>
-  <joint name="joint4" type="revolute">
-    <parent link="link3"/>
-    <child link="wrist_link"/>
-    <origin xyz="0 0 ${link3_length}" rpy="0 0 0"/>
-    <axis xyz="0 1 0"/>
-    <limit lower="-2.0" upper="2.0"
-           effort="5" velocity="1.0"/>
-  </joint>
-  <link name="tool_link">
-    <visual>
-      <origin xyz="0 0 0.04"/>
-      <geometry><box size="0.04 0.04 0.08"/></geometry>
-      <material name="tool_gray">
-        <color rgba="0.85 0.55 0.15 1"/>
-      </material>
-    </visual>
-    <collision>
-      <origin xyz="0 0 0.04"/>
-      <geometry><box size="0.04 0.04 0.08"/></geometry>
-    </collision>
-    <inertial>
-      <origin xyz="0 0 0.04"/>
-      <mass value="0.1"/>
-      <inertia ixx="0.0001" ixy="0" ixz="0"
-               iyy="0.0001" iyz="0" izz="0.0001"/>
-    </inertial>
-  </link>
-  <joint name="joint5" type="revolute">
-    <parent link="wrist_link"/>
-    <child link="tool_link"/>
-    <origin xyz="0 0 0.05" rpy="0 0 0"/>
-    <axis xyz="0 0 1"/>
-    <limit lower="-3.14159" upper="3.14159"
-           effort="5" velocity="1.0"/>
-  </joint>
-  <!-- Fixed placeholder for the gripper attachment -->
-  <link name="gripper_link">
-    <visual>
-      <geometry><box size="0.06 0.025 0.025"/></geometry>
-      <material name="gripper_gray">
-        <color rgba="0.25 0.25 0.27 1"/>
-      </material>
-    </visual>
-    <collision>
-      <geometry><box size="0.06 0.025 0.025"/></geometry>
-    </collision>
-    <inertial>
-      <mass value="0.05"/>
-      <inertia ixx="0.00001" ixy="0" ixz="0"
-               iyy="0.00001" iyz="0" izz="0.00001"/>
-    </inertial>
-  </link>
-  <joint name="gripper_mount" type="fixed">
-    <parent link="tool_link"/>
-    <child link="gripper_link"/>
-    <origin xyz="0 0 0.08" rpy="0 0 0"/>
+          effort="8" velocity="1.0"/>
   </joint>
 </robot>
