Commit message: Changes from 6 to 5dof

File: 5dof-robotic-arm/ros2_ws/src/five_dof_arm/urdf/arm.urdf.xacro (robot description, xacro)
@@ -1,4 +1,4 @@
 <?xml version="1.0"?>
-<robot xmlns:xacro="http://www.ros.org/wiki/xacro" name="six_dof_arm">
+<robot xmlns:xacro="http://www.ros.org/wiki/xacro" name="five_dof_arm">
   <!-- Dimensions are illustrative, in metres. -->
   <xacro:property name="base_height" value="0.08"/>
@@ -12,5 +12,5 @@
       <origin xyz="-0.077 -0.070 0" rpy="0 0 0"/>
       <geometry>
-        <mesh filename="package://six_dof_arm/meshes/Base1.STL"
+        <mesh filename="package://five_dof_arm/meshes/Base1.STL"
               scale="0.001 0.001 0.001"/>
       </geometry>
@@ -20,12 +20,12 @@
   <link name="base2_link">
     <visual>
-      <origin xyz="-0.06 -0.06 0.003" rpy="0 0 0"/>
+      <origin xyz="-0.06 -0.06 0.0" rpy="0 0 0"/>
       <geometry>
-        <mesh filename="package://six_dof_arm/meshes/Base2.STL"
+        <mesh filename="package://five_dof_arm/meshes/Base2.STL"
               scale="0.001 0.001 0.001"/>
       </geometry>
       <material name="base2_blue">
         <color rgba="0.15 0.35 0.8 1.0"/>
-    </material>
+      </material>
     </visual>
   </link>
@@ -33,5 +33,5 @@
     <parent link="base_link"/>
     <child link="base2_link"/>
-    <origin xyz="0 0 0.035" rpy="0 0 0"/>
+    <origin xyz="0 0 0.037" rpy="0 0 0"/>
     <axis xyz="0 0 1"/>
     <limit lower="-3.14159" upper="3.14159"
@@ -43,5 +43,5 @@
       <origin xyz="-0.013 -0.022 -0.008" rpy="0 0 0"/>
       <geometry>
-        <mesh filename="package://six_dof_arm/meshes/Link1.STL"
+        <mesh filename="package://five_dof_arm/meshes/Link1.STL"
               scale="0.001 0.001 0.001"/>
       </geometry>
@@ -51,5 +51,5 @@
     <parent link="base2_link"/>
     <child link="link1"/>
-    <origin xyz="0 0 0.025" rpy="0 0 0"/>
+    <origin xyz="0 0 0.028" rpy="0 0 0"/>
     <axis xyz="0 1 0"/>
     <limit lower="-1.5708" upper="1.5708"
@@ -59,7 +59,7 @@
   <link name="link2">
     <visual>
-      <origin xyz="-0.0148 -0.0145 -0.009" rpy="0 0 0"/>
+      <origin xyz="-0.0148 -0.0145 -0.008" rpy="0 0 0"/>
       <geometry>
-        <mesh filename="package://six_dof_arm/meshes/Link2.STL"
+        <mesh filename="package://five_dof_arm/meshes/Link2.STL"
               scale="0.001 0.001 0.001"/>
       </geometry>
@@ -72,4 +72,22 @@
     <parent link="link1"/>
     <child link="link2"/>
+    <origin xyz="0 0 0.101" rpy="0 0 0"/>
+    <axis xyz="0 1 0"/>
+    <limit lower="-2.0" upper="2.0"
+          effort="8" velocity="1.0"/>
+  </joint>
+  <!-- Joint 4: second arm -->
+  <link name="link3">
+    <visual>
+      <origin xyz="-0.014 -0.016 -0.008" rpy="0 0 0"/>
+      <geometry>
+        <mesh filename="package://five_dof_arm/meshes/Link3.STL"
+              scale="0.001 0.001 0.001"/>
+      </geometry>
+    </visual>
+  </link>
+  <joint name="joint4" type="revolute">
+    <parent link="link2"/>
+    <child link="link3"/>
     <origin xyz="0 0 0.095" rpy="0 0 0"/>
     <axis xyz="0 1 0"/>
@@ -77,3 +95,24 @@
           effort="8" velocity="1.0"/>
   </joint>
+  <!-- Joint 5: End point -->
+  <link name="link4">
+    <visual>
+      <origin xyz="-0.0135 -0.0135 0" rpy="0 0 0"/>
+      <geometry>
+        <mesh filename="package://five_dof_arm/meshes/Link4.STL"
+              scale="0.001 0.001 0.001"/>
+      </geometry>
+      <material name="base2_blue">
+        <color rgba="0.15 0.35 0.8 1.0"/>
+      </material>
+    </visual>
+  </link>
+  <joint name="joint5" type="revolute">
+    <parent link="link3"/>
+    <child link="link4"/>
+    <origin xyz="0 0 0.068" rpy="0 0 0"/>
+    <axis xyz="0 0 1"/>
+    <limit lower="-3.14159" upper="3.14159"
+          effort="10" velocity="1.0"/>
+  </joint>
 </robot>
